File: KiCad/rot-kb/rot-kb.kicad_pcb (KiCad board)
At the start: 2 copper layers, 50 x 100 mm, 30 parts, among them J1 Conn_02x03_Odd_Even, J2 Conn_01x04_Female, J3 Conn_01x03, P1 Digital, P2 Analog, P3 CONN_01X01, P4 CONN_01X01, P5 CONN_01X01, P6 CONN_01X01, P7 ST-TF-003A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

Commit message: mouse mode
Parts:
- removed J3: Conn_01x03, Connector_Phoenix_MC:PhoenixContact_MCV_1,5_3-G-3.81_1x03_P3.81mm_Vertical
- added R2: 10k, Resistor_SMD:R_0805_2012Metric, F.Cu at (148.3, 73.1)
- added R3: 10k, Resistor_SMD:R_0805_2012Metric, F.Cu at (148.3, 91.2)
- added R4: 10k, Resistor_SMD:R_0805_2012Metric, F.Cu at (148.3, 98.8)
- added SW5: SW_DIP_x03, Button_Switch_THT:SW_DIP_SPSTx03_Slide_9.78x9.8mm_W7.62mm_P2.54mm, F.Cu at (157.2, 35.3)
- moved R1 23.6 mm to (148.3, 95.5), turned to 0 degrees
Connections:
- net /A4 renamed Net-(P2-Pad10)
- P2 pad 11: /A3 -> inc4
- P2 pad 12: /A2 -> mouse
- P2 pad 9: /A5 -> rflip
- R1 pad 2: MISO -> inc4
Routing:
- net mouse: track 0.00 -> 70.2 mm
- net inc4: track 0.00 -> 64.3 mm
- net rflip: track 0.00 -> 54.1 mm
- net +3V3: track 123.4 -> 104.0 mm
- net /Vin: track 67.2 -> 60.3 mm
Other:
- board text added: "Flip"
- board text added: "Mouse"
- board text added: "inc4"
- board text removed: "Vin"
