File: KiCad/rot-kb/rot-kb.sch (KiCad schematic (older format))
At the start: 30 parts, among them J1 Conn_02x03_Odd_Even, J2 Conn_01x04_Female, J3 Conn_01x03, P1 Digital, P2 Analog, P3 CONN_01X01, P4 CONN_01X01, P5 CONN_01X01, P6 CONN_01X01, P7 ST-TF-003A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

Commit message: mouse mode
Parts:
- removed J3: Conn_01x03, Connector_Phoenix_MC:PhoenixContact_MCV_1,5_3-G-3.81_1x03_P3.81mm_Vertical, symbol Connector_Generic:Conn_01x03
- added R2, R3, R4: 10k, Resistor_SMD:R_0805_2012Metric, symbol Device:R_US
- added SW5: SW_DIP_x03, Button_Switch_THT:SW_DIP_SPSTx03_Slide_9.78x9.8mm_W7.62mm_P2.54mm, symbol Switch:SW_DIP_x03
Connections:
- net labels added: inc4, mouse, rflip
- net labels removed: A4, A5
- wire segments 53 -> 52
- no-connect marks 10 -> 11
Other:
- moved on the sheet: R1
Changed lines of the file:
@@
 Text Label 10650 2250 0    60   ~ 0
 A3
-Text Label 10650 2150 0    60   ~ 0
-A4
-Text Label 10650 2050 0    60   ~ 0
-A5
 NoConn ~ 10150 1950
 NoConn ~ 10150 1850
@@
 	10150 1350 10650 1350
 Wire Wire Line
-	10650 2050 10150 2050
-Wire Wire Line
-	10150 2150 10650 2150
-Wire Wire Line
-	10650 2250 10150 2250
-Wire Wire Line
 	10150 2650 10650 2650
 Wire Wire Line
@@
 	1    0    0    -1
 $EndComp
-$Comp
-L Device:R_US R1
-U 1 1 5EAB7A01
-P 5950 2400
-F 0 "R1" H 6018 2446 50  0000 L CNN
-F 1 "10k" H 6018 2355 50  0000 L CNN
-F 2 "Resistor_SMD:R_0805_2012Metric" V 5990 2390 50  0001 C CNN
-F 3 "~" H 5950 2400 50  0001 C CNN
-	1    5950 2400
-	1    0    0    -1
-$EndComp
 Text GLabel 5850 1700 3    50   Input ~ 0
 MISO
 Text GLabel 5950 2550 3    50   Input ~ 0
 MISO
-$Comp
-L power:+3V3 #PWR0110
-U 1 1 5EAB9327
-P 5950 2250
-F 0 "#PWR0110" H 5950 2100 50  0001 C CNN
-F 1 "+3.3V" H 5950 2390 28  0000 C CNN
-F 2 "" H 5950 2250 50  0000 C CNN
-F 3 "" H 5950 2250 50  0000 C CNN
-	1    5950 2250
-	1    0    0    -1
-$EndComp
 Text GLabel 5550 1700 3    50   Input ~ 0
 SCK
@@
 NoConn ~ 9350 1650
 $Comp
-L Connector_Generic:Conn_01x03 J3
-U 1 1 5EB6BBD5
-P 7200 3050
-F 0 "J3" H 7280 3092 50  0000 L CNN
-F 1 "Conn_01x03" H 7280 3001 50  0000 L CNN
-F 2 "Connector_Phoenix_MC:PhoenixContact_MCV_1,5_3-G-3.81_1x03_P3.81mm_Vertical" H 7200 3050 50  0001 C CNN
-F 3 "~" H 7200 3050 50  0001 C CNN
-	1    7200 3050
-	1    0    0    -1
-$EndComp
-$Comp
-L power:GND #PWR0111
-U 1 1 5EB6C347
-P 7000 2950
-F 0 "#PWR0111" H 7000 2700 50  0001 C CNN
-F 1 "GND" V 7005 2822 50  0000 R CNN
-F 2 "" H 7000 2950 50  0001 C CNN
-F 3 "" H 7000 2950 50  0001 C CNN
-	1    7000 2950
-	0    1    1    0
-$EndComp
-$Comp
-L power:+3V3 #PWR0112
-U 1 1 5EB6CA0E
-P 7000 3150
-F 0 "#PWR0112" H 7000 3000 50  0001 C CNN
-F 1 "+3.3V" H 7000 3290 28  0000 C CNN
-F 2 "" H 7000 3150 50  0000 C CNN
-F 3 "" H 7000 3150 50  0000 C CNN
-	1    7000 3150
-	0    -1   -1   0
-$EndComp
-Text Label 6650 3050 2    60   ~ 0
-Vin
-Wire Wire Line
-	7000 3050 6650 3050
-$Comp
 L Device:C C1
 U 1 1 5EB8F30D
@@
 Text GLabel 8750 2750 0    50   Input ~ 0
 ecn4
+$Comp
+L Device:R_US R2
+U 1 1 5F223F73
+P 5950 2400
+F 0 "R2" H 6018 2446 50  0000 L CNN
+F 1 "10k" H 6018 2355 50  0000 L CNN
+F 2 "Resistor_SMD:R_0805_2012Metric" V 5990 2390 50  0001 C CNN
+F 3 "~" H 5950 2400 50  0001 C CNN
+	1    5950 2400
+	1    0    0    -1
+$EndComp
+$Comp
+L power:+3V3 #PWR05
+U 1 1 5F224999
+P 5950 2250
+F 0 "#PWR05" H 5950 2100 50  0001 C CNN
+F 1 "+3.3V" H 5950 2390 28  0000 C CNN
+F 2 "" H 5950 2250 50  0000 C CNN
+F 3 "" H 5950 2250 50  0000 C CNN
+	1    5950 2250
+	1    0    0    -1
+$EndComp
+$Comp
+L Device:R_US R1
+U 1 1 5EAB7A01
+P 13200 3050
+F 0 "R1" H 13268 3096 50  0000 L CNN
+F 1 "10k" H 13268 3005 50  0000 L CNN
+F 2 "Resistor_SMD:R_0805_2012Metric" V 13240 3040 50  0001 C CNN
+F 3 "~" H 13200 3050 50  0001 C CNN
+	1    13200 3050
+	1    0    0    -1
+$EndComp
+$Comp
+L power:+3V3 #PWR0110
+U 1 1 5EAB9327
+P 13000 2800
+F 0 "#PWR0110" H 13000 2650 50  0001 C CNN
+F 1 "+3.3V" H 13000 2940 28  0000 C CNN
+F 2 "" H 13000 2800 50  0000 C CNN
+F 3 "" H 13000 2800 50  0000 C CNN
+	1    13000 2800
+	1    0    0    -1
+$EndComp
+$Comp
+L Device:R_US R3
+U 1 1 5F230F09
+P 13000 2950
+F 0 "R3" H 13068 2996 50  0000 L CNN
+F 1 "10k" H 13068 2905 50  0000 L CNN
+F 2 "Resistor_SMD:R_0805_2012Metric" V 13040 2940 50  0001 C CNN
+F 3 "~" H 13000 2950 50  0001 C CNN
+	1    13000 2950
+	-1   0    0    1
+$EndComp
+Text GLabel 12900 3100 3    50   Input ~ 0
+rflip
+Text GLabel 10150 2050 2    50   Input ~ 0
+rflip
+Text GLabel 13100 3200 3    50   Input ~ 0
+inc4
+Text GLabel 10150 2250 2    50   Input ~ 0
+inc4
+NoConn ~ 10150 2150
+$Comp
+L Switch:SW_DIP_x03 SW5
+U 1 1 5F243952
+P 12500 3300
+F 0 "SW5" H 12500 3767 50  0000 C CNN
+F 1 "SW_DIP_x03" H 12500 3676 50  0000 C CNN
+F 2 "Button_Switch_THT:SW_DIP_SPSTx03_Slide_9.78x9.8mm_W7.62mm_P2.54mm" H 12500 3300 50  0001 C CNN
+F 3 "~" H 12500 3300 50  0001 C CNN
+	1    12500 3300
+	1    0    0    -1
+$EndComp
+Wire Wire Line
+	12800 3100 13000 3100
+Wire Wire Line
+	13200 3200 12800 3200
+$Comp
+L Device:R_US R4
+U 1 1 5F24B293
+P 13450 3150
+F 0 "R4" H 13518 3196 50  0000 L CNN
+F 1 "10k" H 13518 3105 50  0000 L CNN
+F 2 "Resistor_SMD:R_0805_2012Metric" V 13490 3140 50  0001 C CNN
+F 3 "~" H 13450 3150 50  0001 C CNN
+	1    13450 3150
+	1    0    0    -1
+$EndComp
+Wire Wire Line
+	12800 3300 13450 3300
+$Comp
+L power:+3V3 #PWR0115
+U 1 1 5F24E97C
+P 13200 2900
+F 0 "#PWR0115" H 13200 2750 50  0001 C CNN
+F 1 "+3.3V" H 13200 3040 28  0000 C CNN
+F 2 "" H 13200 2900 50  0000 C CNN
+F 3 "" H 13200 2900 50  0000 C CNN
+	1    13200 2900
+	1    0    0    -1
+$EndComp
+$Comp
+L power:+3V3 #PWR0118
+U 1 1 5F24EEA5
+P 13450 3000
+F 0 "#PWR0118" H 13450 2850 50  0001 C CNN
+F 1 "+3.3V" H 13450 3140 28  0000 C CNN
+F 2 "" H 13450 3000 50  0000 C CNN
+F 3 "" H 13450 3000 50  0000 C CNN
+	1    13450 3000
+	1    0    0    -1
+$EndComp
+Text GLabel 13300 3300 3    50   Input ~ 0
+mouse
+$Comp
+L power:GND #PWR0119
+U 1 1 5F25105C
+P 12200 3300
+F 0 "#PWR0119" H 12200 3050 50  0001 C CNN
+F 1 "GND" H 12200 3150 50  0000 C CNN
+F 2 "" H 12200 3300 50  0000 C CNN
+F 3 "" H 12200 3300 50  0000 C CNN
+	1    12200 3300
+	0    1    1    0
+$EndComp
+$Comp
+L power:GND #PWR0120
+U 1 1 5F251A00
+P 12200 3200
+F 0 "#PWR0120" H 12200 2950 50  0001 C CNN
+F 1 "GND" H 12200 3050 50  0000 C CNN
+F 2 "" H 12200 3200 50  0000 C CNN
+F 3 "" H 12200 3200 50  0000 C CNN
+	1    12200 3200
+	0    1    1    0
+$EndComp
+$Comp
+L power:GND #PWR0121
+U 1 1 5F251BE5
+P 12200 3100
+F 0 "#PWR0121" H 12200 2850 50  0001 C CNN
+F 1 "GND" H 12200 2950 50  0000 C CNN
+F 2 "" H 12200 3100 50  0000 C CNN
+F 3 "" H 12200 3100 50  0000 C CNN
+	1    12200 3100
+	0    1    1    0
+$EndComp
+Text GLabel 10950 2350 2    50   Input ~ 0
+mouse
 $EndSCHEMATC
